File: Sump-pcb/sump-pcb.sch (KiCad schematic (older format))
At the start: 11 parts

Commit message: sump pcb now 2x1 with 2x mosfets
Parts:
- removed P? (x2): CONN_01X04, symbol CONN_01X04
- added 10k1, 10k2: R, Resistors_SMD:R_0805, symbol R
- added D1: LED, LEDs:LED-0805, symbol LED
- added P1: Vin, Pin_Headers:Pin_Header_Straight_1x02, symbol CONN_01X02
- added P4: I2C, Pin_Headers:Pin_Header_Straight_1x04, symbol CONN_01X04
- added P5: GPIO, Pin_Headers:Pin_Header_Straight_1x04, symbol CONN_01X04
- added Q1, Q2: 3401P, Housings_SOT-23_SOT-143_TSOT-6:SOT-23, symbol IRF9540N
- C1, C2, C3: renamed from C?; footprint (none) -> Capacitors_SMD:C_0805
- P2: renamed from P?; value CONN_01X06 -> ISP; footprint (none) -> Pin_Headers:Pin_Header_Straight_1x06
- P3: renamed from P?; value CONN_01X04 -> sonar; footprint (none) -> Pin_Headers:Pin_Header_Straight_1x04
- P6: renamed from P?; footprint (none) -> Pin_Headers:Pin_Header_Straight_2x03
- U1: renamed from U?; footprint (none) -> Housings_SOT-23_SOT-143_TSOT-6:SOT-23_Handsoldering
- U2: renamed from U?; footprint MODULE -> RFM69BreakoutBoardFootPrints:RFM69HW
- gave numbers to parts that had none: 1
Connections:
- net labels added: I2Cpower
- wire segments 98 -> 149
